File: hardware/PCB air_controller/PCB air_controller 2.kicad_pcb (KiCad board)
At the start: 2 copper layers, 35 parts, among them J1 Conn_01x02, J2 Conn_01x02, J3 Conn_01x02, J4 Conn_01x05, J5 Conn_01x08, Q1 MMBT2222L, Q2 MMBT2222L, Q3 MMBT2222L, Q4 s8550, Q5 s8550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

Commit message: hardware :: fix brd
Parts:
- U3: moved to B.Cu
- moved U3 34.8 mm to (46.2, 28.6)
- moved Q5 21.6 mm to (44.7, 54.9), turned to 180 degrees
Routing:
- net cs: track 68.7 -> 24.9 mm, vias 2 -> 0
- net black_light: track 29.7 -> 62.9 mm, vias 0 -> 2
- net GND: track 37.7 -> 69.0 mm, vias 0 -> 4
- net sda: track 47.1 -> 63.2 mm
- net ao: track 24.1 -> 38.0 mm
- net en2_a: track 45.7 -> 57.7 mm
- net lcd_reset: track 24.7 -> 31.6 mm
- net +5V: track 174.1 -> 168.0 mm
- net en2_b: track 38.8 -> 43.1 mm
- net Net-(Q5-Pad3): track 2.45 -> 4.81 mm
- net (no net): track 0.00 -> 2.21 mm
- net sck: track 30.7 -> 29.4 mm, vias 2 -> 0
- net en2_btn: track 53.8 -> 54.0 mm, vias 9 -> 0
