File: hardware/PCB air_controller/PCB air_controller.sch (KiCad schematic (older format))
At the start: 35 parts, among them J1 Conn_01x02, J2 Conn_01x02, J3 Conn_01x02, J4 Conn_01x05, J5 Conn_01x08, Q1 MMBT2222L, Q3 MMBT2222L, Q4 s8550, Q5 s8550, SW1 Rotary_Encoder_Switch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

Commit message: hardware :: fix brd
Parts:
- gave numbers to parts that had none: 6
Changed lines of the file:
@@
 	4850 1350 5375 1350
 $Comp
-L Transistor_BJT:BC807 Q?
+L Transistor_BJT:BC807 Q6
 U 1 1 5D1EC0C6
 P 5050 3875
-F 0 "Q?" H 5241 3921 50  0000 L CNN
+F 0 "Q6" H 5241 3921 50  0000 L CNN
 F 1 "s8550" H 5241 3830 50  0000 L CNN
 F 2 "Package_TO_SOT_SMD:SOT-23" H 5250 3800 50  0001 L CIN
@@
 $EndComp
 $Comp
-L power:+12V #PWR?
+L power:+12V #PWR0101
 U 1 1 5D1EC0CC
 P 5150 3675
-F 0 "#PWR?" H 5150 3525 50  0001 C CNN
+F 0 "#PWR0101" H 5150 3525 50  0001 C CNN
 F 1 "+12V" H 5165 3848 50  0000 C CNN
 F 2 "" H 5150 3675 50  0001 C CNN
@@
 $EndComp
 $Comp
-L Transistor_BJT:BC807 Q?
+L Transistor_BJT:BC807 Q7
 U 1 1 5D1EF4CB
 P 5050 4800
-F 0 "Q?" H 5241 4846 50  0000 L CNN
+F 0 "Q7" H 5241 4846 50  0000 L CNN
 F 1 "s8550" H 5241 4755 50  0000 L CNN
 F 2 "Package_TO_SOT_SMD:SOT-23" H 5250 4725 50  0001 L CIN
@@
 $EndComp
 $Comp
-L power:+12V #PWR?
+L power:+12V #PWR0102
 U 1 1 5D1EF4D1
 P 5150 4600
-F 0 "#PWR?" H 5150 4450 50  0001 C CNN
+F 0 "#PWR0102" H 5150 4450 50  0001 C CNN
 F 1 "+12V" H 5165 4773 50  0000 C CNN
 F 2 "" H 5150 4600 50  0001 C CNN
@@
 	5150 4125 5225 4125
 $Comp
-L Device:R_Small R?
+L Device:R_Small R11
 U 1 1 5D1FFD15
 P 4750 3875
-F 0 "R?" H 4691 3829 50  0000 R CNN
+F 0 "R11" H 4691 3829 50  0000 R CNN
 F 1 "R_Small" H 4691 3920 50  0000 R CNN
 F 2 "Resistor_SMD:R_0805_2012Metric" H 4750 3875 50  0001 C CNN
@@
 $EndComp
 $Comp
-L Device:R_Small R?
+L Device:R_Small R13
 U 1 1 5D202CF4
 P 4750 4800
-F 0 "R?" H 4691 4754 50  0000 R CNN
+F 0 "R13" H 4691 4754 50  0000 R CNN
 F 1 "R_Small" H 4691 4845 50  0000 R CNN
 F 2 "Resistor_SMD:R_0805_2012Metric" H 4750 4800 50  0001 C CNN
@@
 $EndComp
 $Comp
-L Device:R_Small R?
+L Device:R_Small R10
 U 1 1 5D204E85
 P 4625 5850
-F 0 "R?" H 4566 5804 50  0000 R CNN
+F 0 "R10" H 4566 5804 50  0000 R CNN
 F 1 "R_Small" H 4566 5895 50  0000 R CNN
 F 2 "Resistor_SMD:R_0805_2012Metric" H 4625 5850 50  0001 C CNN
@@
 $EndComp
 $Comp
-L Transistor_BJT:MMBT3904 Q?
+L Transistor_BJT:MMBT3904 Q2
 U 1 1 5D210700
 P 4550 4075
-F 0 "Q?" H 4741 4121 50  0000 L CNN
+F 0 "Q2" H 4741 4121 50  0000 L CNN
 F 1 "MMBT2222L" H 4741 4030 50  0000 L CNN
 F 2 "Package_TO_SOT_SMD:SOT-23" H 4750 4000 50  0001 L CIN
@@
 $EndComp
 $Comp
-L power:GND #PWR?
+L power:GND #PWR0103
 U 1 1 5D210706
 P 4650 4275
-F 0 "#PWR?" H 4650 4025 50  0001 C CNN
+F 0 "#PWR0103" H 4650 4025 50  0001 C CNN
 F 1 "GND" H 4655 4102 50  0000 C CNN
 F 2 "" H 4650 4275 50  0001 C CNN
